File: pcb/Si5351ABreakout.sch (KiCad schematic (older format))
At the start: 23 parts, among them J1 Power/Data, J10 Osc Power, J2 PS SEL, J3 3.3V SEL, J4 SMA-F, J5 SMA-F, J6 SMA-F, J7 CLK0, J8 CLK1, J9 CLK2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

Commit message: Rev D PCB changes
Parts:
- removed J10: Osc Power, symbol JUMPER
- added R5, R6, R7, R8: 0, Resistors_SMD:R_0805, symbol R
- C1, C2, C3, C4: footprint (none) -> Capacitors_SMD:C_0805
- J1: footprint (none) -> Pin_Headers:Pin_Header_Straight_1x05_Pitch2.54mm
- J2, J3: footprint (none) -> Pin_Headers:Pin_Header_Straight_1x03_Pitch2.54mm
- J4, J5, J6: footprint (none) -> EtherkitKicadLibrary:SMA-ENDLAUNCH
- J7, J8, J9: footprint (none) -> Pin_Headers:Pin_Header_Straight_1x02_Pitch2.54mm
- Q1, Q2: footprint (none) -> EtherkitKicadLibrary:SOT23-2N7002
- R1, R2, R3, R4: footprint (none) -> Resistors_SMD:R_0805
- U1: footprint (none) -> EtherkitKicadLibrary:SOT23-5
- U2: footprint MODULE -> EtherkitKicadLibrary:MSOP-10
- X1: value FOX924B-25.000 or ECS-250-8-30B-CKM -> ASTX-H11-25.000MHZ-T or ECS-250-8-30B-CKM; footprint (none) -> EtherkitKicadLibrary:ASTX-H11-25.000MHZ-T
Connections:
- net +3.3VREG: now also X1.4 (VDD), R5.1
- net GND: now also R6.2, R8.2
- net at U2.2 (XA): now also R7.2, R8.1; no longer X1.3 (OUT)
- net at U2.3 (XB), X1.1 (OE): now also R5.2
- new net: R6.1, R7.1, X1.3 (OUT)
Other:
- moved on the sheet: X1

Commit message: Rev D Update
Parts:
- added R6: 0, Resistors_SMD:R_0805, symbol R
- renumbered R6 to R7, R7 to R8, R8 to R9
Connections:
- net +3.3VREG: now also R6.1; no longer R5.1, X1.4 (VDD)
- new net: R5.1, R6.2, X1.4 (VDD)
Changed lines of the file:
@@
 EESchema Schematic File Version 2
-LIBS:Si5351ABreakout-rescue
 LIBS:EtherkitKicadLibrary
 LIBS:power
@@
 Sheet 1 1
 Title "Si5351A Breakout"
-Date "2017-01-28"
+Date "2017-07-16"
 Rev "D"
 Comp "Etherkit"
@@
 Comment2 ""
 Comment3 ""
-Comment4 "Creative Commons Licence CC-BY-SA"
+Comment4 "Creative Commons License CC-BY-SA"
 $EndDescr
 $Comp
@@
 L +3.3VREG #PWR018
 U 1 1 53D57D6D
-P 4055 2665
-F 0 "#PWR018" H 4055 2625 30  0001 C CNN
-F 1 "+3.3VREG" H 4055 2775 30  0000 C CNN
-F 2 "" H 4055 2665 60  0000 C CNN
-F 3 "" H 4055 2665 60  0000 C CNN
-	1    4055 2665
+P 4055 2365
+F 0 "#PWR018" H 4055 2325 30  0001 C CNN
+F 1 "+3.3VREG" H 4055 2475 30  0000 C CNN
+F 2 "" H 4055 2365 60  0000 C CNN
+F 3 "" H 4055 2365 60  0000 C CNN
+	1    4055 2365
 	1    0    0    -1
 $EndComp
@@
 Connection ~ 4055 2720
 $Comp
-L R R6
+L R R7
 U 1 1 588D31D1
 P 4480 3380
-F 0 "R6" H 4600 3420 50  0000 C CNN
+F 0 "R7" H 4600 3420 50  0000 C CNN
 F 1 "0" H 4580 3340 50  0001 C CNN
 F 2 "Resistors_SMD:R_0805" H 4480 3380 60  0001 C CNN
@@
 $EndComp
 $Comp
-L R R8
+L R R9
 U 1 1 588D333B
 P 4880 3380
-F 0 "R8" H 5000 3420 50  0000 C CNN
+F 0 "R9" H 5000 3420 50  0000 C CNN
 F 1 "0" H 4980 3340 50  0001 C CNN
 F 2 "Resistors_SMD:R_0805" H 4880 3380 60  0001 C CNN
@@
 $EndComp
 $Comp
-L R R7
+L R R8
 U 1 1 588D362C
 P 4680 3230
-F 0 "R7" V 4775 3225 50  0000 C CNN
+F 0 "R8" V 4775 3225 50  0000 C CNN
 F 1 "0" V 4780 3120 50  0001 C CNN
 F 2 "Resistors_SMD:R_0805" H 4680 3230 60  0001 C CNN
@@
 Wire Wire Line
 	6690 3525 6855 3525
+$Comp
+L R R6
+U 1 1 58A9E9AD
+P 4055 2515
+F 0 "R6" H 4175 2555 50  0000 C CNN
+F 1 "0" H 4155 2475 50  0000 C CNN
+F 2 "Resistors_SMD:R_0805" H 4055 2515 60  0001 C CNN
+F 3 "" H 4055 2515 60  0000 C CNN
+	1    4055 2515
+	1    0    0    -1
+$EndComp
 $EndSCHEMATC
