File: pcb/Si5351ABreakout_conflict-20150214-094747.sch (KiCad schematic (older format))
At the start: 23 parts, among them J1 Power/Data, J10 Osc Power, J2 PS SEL, J3 3.3V SEL, J4 SMA-F, J5 SMA-F, J6 SMA-F, J7 CLK0, J8 CLK1, J9 CLK2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

Commit message: Update schematic, PCB 50 ohm output traces
Parts:
- C2: value 10n -> 100n
Changed lines of the file:
@@
 LIBS:valves
 LIBS:Si5351ABreakout-cache
-EELAYER 24 0
+EELAYER 25 0
 EELAYER END
 $Descr USLetter 11000 8500
@@
 Sheet 1 1
 Title "Si5351A Breakout"
-Date "15 Jan 2015"
+Date "Sat 14 Feb 2015"
 Rev "C"
 Comp "Etherkit"
@@
 P 1975 1835
 F 0 "C2" H 2125 1870 50  0000 C CNN
-F 1 "10n" H 2155 1790 50  0000 C CNN
+F 1 "100n" H 2168 1790 50  0000 C CNN
 F 2 "" H 1975 1835 60  0000 C CNN
 F 3 "" H 1975 1835 60  0000 C CNN
