File: pcb/Si5351ABreakout.kicad_pcb (KiCad board)
At the start: 2 copper layers, 30 x 50 mm, 128 parts, among them J1 Power/Data, J10 Osc Power, J2 PS SEL, J3 3.3V SEL, J4 SMA-F, J5 SMA-F, J6 SMA-F, J7 CLK0, J8 CLK1, J9 CLK2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

Commit message: Rev D PCB changes
Parts:
- removed J10: Osc Power, EtherkitKicadLibrary:SIL-2
- removed the VIA at (108.1, 86.2)
- removed the VIA at (108.1, 85.2)
- removed the VIA at (114.3, 91.9)
- removed the VIA at (114.3, 91.0)
- added R5: 0, Resistors_SMD:R_0805, F.Cu at (109.5, 80.8)
- added R6: 0, Resistors_SMD:R_0805, F.Cu at (115.6, 80.8)
- added R7: 0, Resistors_SMD:R_0805, F.Cu at (114.2, 84.3)
- added R8: 0, Resistors_SMD:R_0805, F.Cu at (112.1, 84.3)
- added REF**: Fiducial_1mm_Dia_2.54mm_Outer_CopperTop, Fiducials:Fiducial_1mm_Dia_2.54mm_Outer_CopperTop, F.Cu at (125.0, 93.0)
- added REF**: Fiducial_1mm_Dia_2.54mm_Outer_CopperTop, Fiducials:Fiducial_1mm_Dia_2.54mm_Outer_CopperTop, F.Cu at (106.5, 93.0)
- added REF**: Fiducial_1mm_Dia_2.54mm_Outer_CopperTop, Fiducials:Fiducial_1mm_Dia_2.54mm_Outer_CopperTop, F.Cu at (125.0, 56.2)
- C1, C3, C4: footprint EtherkitKicadLibrary:SM0805 -> Capacitors_SMD:C_0805
- C2: value 10n -> 100n; footprint EtherkitKicadLibrary:SM0805 -> Capacitors_SMD:C_0805
- J1: footprint EtherkitKicadLibrary:SIL-5 -> Pin_Headers:Pin_Header_Straight_1x05_Pitch2.54mm
- J2, J3: footprint EtherkitKicadLibrary:SIL-3 -> Pin_Headers:Pin_Header_Straight_1x03_Pitch2.54mm
- J7, J8, J9: footprint EtherkitKicadLibrary:SIL-2 -> Pin_Headers:Pin_Header_Straight_1x02_Pitch2.54mm
- R1, R2, R3, R4: footprint EtherkitKicadLibrary:SM0805 -> Resistors_SMD:R_0805
- U2: value Si5351A -> Si5351A-B
- X1: value FOX924B-25.000 or ECS-250-8-30B-CKM -> ASTX-H11-25.000MHZ-T or ECS-250-8-30B-CKM; footprint EtherkitKicadLibrary:ECS-250-8-30B-CKM -> EtherkitKicadLibrary:ASTX-H11-25.000MHZ-T
- moved J1 6.35 mm to (102.7, 58.8), turned to 0 degrees
- moved J2 2.54 mm to (102.7, 73.8), turned to 0 degrees
- moved J3 2.53 mm to (110.9, 58.4), turned to 90 degrees
- moved J8 1.30 mm to (122.5, 75.0), turned to 0 degrees
- moved J9 1.30 mm to (122.5, 87.0), turned to 0 degrees
- moved J7 1.20 mm to (122.5, 63.0), turned to 0 degrees
- moved X1 0.78 mm to (112.7, 80.8)
Connections:
- U2 pad 2: Net-(U2-Pad2) -> Net-(R7-Pad2)
- X1 pad 3: Net-(U2-Pad2) -> Net-(R6-Pad1)
- X1 pad 4: Net-(J10-Pad2) -> +3.3VREG
Routing:
- net Net-(U2-Pad2): track 9.20 -> 0.00 mm
- net Net-(J10-Pad2): track 7.79 -> 0.00 mm
- net Net-(R6-Pad1): track 0.00 -> 7.34 mm
- net Net-(R7-Pad2): track 0.00 -> 4.56 mm
- net +3.3VREG: track 66.1 -> 70.2 mm
- net Net-(R5-Pad2): track 6.00 -> 8.64 mm
- net Net-(Q1-Pad1): track 24.4 -> 26.0 mm
Other:
- board text added: "I2C Address: 0x60 (7-bit)"
- board text added: "Rev D"
- board text added: "etherkit.com 2017"
- board text removed: "I2C Address: 0x60 (7-bit) 0xC0 (8-bit write) 0xC1 (8-bit read)"
- board text removed: "OSC PWR"
- board text removed: "Rev C"
- board text removed: "etherkit.com 2015"

Commit message: Rev D Update
Parts:
- added R9: 0, Resistors_SMD:R_0805, F.Cu at (112.2, 84.3)
- moved R6 9.10 mm to (106.5, 80.8)
- moved R7 3.83 mm to (115.7, 80.8)
- moved R8 2.05 mm to (114.2, 84.3), turned to 270 degrees
Connections:
- R5 pad 1: +3.3VREG -> Net-(R5-Pad1)
- R6 pad 1: Net-(R6-Pad1) -> +3.3VREG
- R6 pad 2: GND -> Net-(R5-Pad1)
- R7 pad 1: Net-(R6-Pad1) -> Net-(R7-Pad1)
- R7 pad 2: Net-(R7-Pad2) -> GND
- R8 pad 1: Net-(R7-Pad2) -> Net-(R7-Pad1)
- R8 pad 2: GND -> Net-(R8-Pad2)
- U2 pad 2: Net-(R7-Pad2) -> Net-(R8-Pad2)
- X1 pad 3: Net-(R6-Pad1) -> Net-(R7-Pad1)
- X1 pad 4: +3.3VREG -> Net-(R5-Pad1)
Routing:
- net Net-(R7-Pad1): track 0.00 -> 7.34 mm
- net Net-(R6-Pad1): track 7.34 -> 0.00 mm
- net Net-(R5-Pad1): track 0.00 -> 6.48 mm
- net Net-(R7-Pad2): track 4.56 -> 0.00 mm
- net Net-(R8-Pad2): track 0.00 -> 4.46 mm
- net +3.3VREG: track 70.2 -> 66.8 mm
Other:
- board text added: "I2C Addr: 0x60 (7-bit)"
- board text removed: "I2C Address: 0x60 (7-bit)"
